File: PCB/_autosave-numberpad.kicad_pcb (KiCad board)
At the start: 2 copper layers, 97 x 124.9 mm, 57 parts, among them J1 Light_Sensor, J2 Rotary_Encoder, J3 Screen_Connector, J4 FingerPrint, SW0 0, SW1 ., SW10 8, SW11 9, SW12 +, SW13 num_lock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

Commit message: update screen support now display information for the screen + brightness.
Parts:
- added D34: SK6812MINI, LED_SMD:LED_SK6812MINI_PLCC4_3.5x3.5mm_P1.75mm, F.Cu at (96.9, 75.9)
- moved D17 37.8 mm to (114.9, 75.4)
